Commit message: rotated 4 corner propellers to match last semester design

File: controls/Kwad.xacro (robot description, xacro)
@@ -271,5 +271,5 @@
 		<parent link="base_link2" />
 		<child link="prop_front_right" />
-		<origin xyz="${prop_loc - 0.01} ${prop_loc - 0.01} 0.021" rpy="0 0 0"/>
+		<origin xyz="${prop_loc - 0.01} ${prop_loc - 0.01} 0.021" rpy="${pi_value/2} 0 ${-pi_value/4}"/>
 		<axis xyz="0 0 1" />
 	</joint>
@@ -279,5 +279,5 @@
 		<parent link="base_link1" />
 		<child link="prop_front_left" />
-		<origin xyz="${-prop_loc + 0.01} ${prop_loc - 0.01} 0.021" rpy="0 0 0" />
+		<origin xyz="${-prop_loc + 0.01} ${prop_loc - 0.01} 0.021" rpy="${pi_value/2} 0 ${pi_value/4}" />
 		<axis xyz="0 0 1" />
 	</joint>
@@ -287,5 +287,5 @@
 		<parent link="base_link1" />
 		<child link="prop_back_right" />
-		<origin xyz="${prop_loc - 0.01} ${-prop_loc + 0.01} 0.021" rpy="0 0 0" />
+		<origin xyz="${prop_loc - 0.01} ${-prop_loc + 0.01} 0.021" rpy="${pi_value/2} 0 ${pi_value/4}" />
 		<axis xyz="0 0 1" />
 	</joint>
@@ -295,5 +295,5 @@
 		<parent link="base_link2" />
 		<child link="prop_back_left" />
-		<origin xyz="${-prop_loc + 0.01} ${-prop_loc + 0.01} 0.021" rpy="0 0 0" />
+		<origin xyz="${-prop_loc + 0.01} ${-prop_loc + 0.01} 0.021" rpy="${-pi_value/2} 0 ${-pi_value/4}" />
 		<axis xyz="0 0 1" />
 	</joint>
