Commit message: modified propeller layout to match 2019 model

File: 2020_workspace/src/mate_simulation/urdf/Kwad.xacro (robot description, xacro)
@@ -58,4 +58,38 @@
 	</link>
 <!-- ======================================================== -->
+	<link name="base_link3">
+		<visual>
+			<origin xyz="0 0 0" rpy="0 0 0" />
+			<geometry>
+				<box size="${width} ${length} ${height}" />
+			</geometry>
+			<material name="blue" />
+		</visual>
+		<collision>
+			<origin xyz="0 0 0" rpy="0 0 0" />
+			<geometry>
+				<box size="${width} ${length} ${height}" />
+			</geometry>
+		</collision>
+		<xacro:default_inertial mass="${mass_fr}" p="${pi_value/4}" ix_value="${0.04989/2}" iy_value="${0.04989/2}" iz_value="${0.24057/2}" />
+	</link>
+<!-- ======================================================== -->
+	<link name="base_link4">
+		<visual>
+			<origin xyz="0 0 0" rpy="0 0 ${pi_value/2}" />
+			<geometry>
+				<box size="${width} ${length} ${height}" />
+			</geometry>
+			<material name="green" />
+		</visual>
+		<collision>
+			<origin xyz="0 0 0" rpy="0 0 ${pi_value/2}" />
+			<geometry>
+				<box size="${width} ${length} ${height}" />
+			</geometry>
+		</collision>
+		<xacro:default_inertial mass="${mass_fr}" p="${-pi_value/4}" ix_value="${0.04989/2}" iy_value="${0.04989/2}" iz_value="${0.24057/2}" />
+	</link>
+<!-- ======================================================== -->
 	<link name="plate1">
 		<visual>
@@ -258,6 +292,70 @@
 		<xacro:default_inertial mass="${mass_pr}" p="${0}"  ix_value="${0}" iy_value="${0}" iz_value="${4.42448e-5}" />
 	</link>
-<!-- ======================================================== -->
-	<!-- Define the joint between the arms of the frame -->
+	<link name="prop_front_middle">
+		<visual>
+			<origin xyz="0 0 0" rpy="0 0 0" />
+			<geometry>
+				<box size="${0.03302/3} ${radiusp*0.8} ${0.001}" />
+			</geometry>
+			<material name="black" />
+		</visual>
+		<collision>
+			<origin xyz="0 0 0" rpy="0 0 0" />
+			<geometry>
+				<box size="${0.03302/3} ${radiusp*0.8} ${0.001}" />
+			</geometry>
+		</collision>
+		<xacro:default_inertial mass="${mass_pr}" p="${0}" ix_value="${0}" iy_value="${0}" iz_value="${4.42448e-5}" />
+	</link>
+	<link name="prop_back_middle">
+		<visual>
+			<origin xyz="0 0 0" rpy="0 0 0" />
+			<geometry>
+				<box size="${0.03302/3} ${radiusp*0.8} ${0.001}" />
+			</geometry>
+			<material name="black" />
+		</visual>
+		<collision>
+			<origin xyz="0 0 0" rpy="0 0 0" />
+			<geometry>
+				<box size="${0.03302/3} ${radiusp*0.8} ${0.001}" />
+			</geometry>
+		</collision>
+		<xacro:default_inertial mass="${mass_pr}" p="${0}" ix_value="${0}" iy_value="${0}" iz_value="${4.42448e-5}" />
+	</link>
+	<link name="prop_right_middle">
+		<visual>
+			<origin xyz="0 0 0" rpy="0 0 0" />
+			<geometry>
+				<box size="${0.03302/3} ${radiusp*0.8} ${0.001}" />
+			</geometry>
+			<material name="black" />
+		</visual>
+		<collision>
+			<origin xyz="0 0 0" rpy="0 0 0" />
+			<geometry>
+				<box size="${0.03302/3} ${radiusp*0.8} ${0.001}" />
+			</geometry>
+		</collision>
+		<xacro:default_inertial mass="${mass_pr}" p="${0}" ix_value="${0}" iy_value="${0}" iz_value="${4.42448e-5}" />
+	</link>
+	<link name="prop_left_middle">
+		<visual>
+			<origin xyz="0 0 0" rpy="0 0 0" />
+			<geometry>
+				<box size="${0.03302/3} ${radiusp*0.8} ${0.001}" />
+			</geometry>
+			<material name="black" />
+		</visual>
+		<collision>
+			<origin xyz="0 0 0" rpy="0 0 0" />
+			<geometry>
+				<box size="${0.03302/3} ${radiusp*0.8} ${0.001}" />
+			</geometry>
+		</collision>
+		<xacro:default_inertial mass="${mass_pr}" p="${0}" ix_value="${0}" iy_value="${0}" iz_value="${4.42448e-5}" />
+	</link>
+<!-- ======================================================== -->
+<!-- Define the joint between the arms of the frame -->
 	<joint name="center" type="fixed">
 		<parent link="base_link1" />
@@ -267,5 +365,21 @@
 	</joint>
 <!-- ======================================================== -->
-	<!-- Define joint between prop fr and frame -->
+<!-- Define the joint between the arms of the frame 2 -->
+	<joint name="center2" type="fixed">
+		<parent link="base_link2" />
+		<child link="base_link3" />
+		<origin xyz="0 0 0" rpy="0 0 0"/>
+		<axis xyz="0 0 1" />
+	</joint>
+<!-- ======================================================== -->
+<!-- Define the joint between the arms of the frame 3 -->
+	<joint name="center3" type="fixed">
+		<parent link="base_link3" />
+		<child link="base_link4" />
+		<origin xyz="0 0 0" rpy="0 0 0"/>
+		<axis xyz="0 0 1" />
+	</joint>
+<!-- ======================================================== -->
+<!-- Define joint between prop fr and frame -->
 	<joint name="joint_front_right_prop" type="continuous">
 		<parent link="base_link2" />
@@ -275,5 +389,5 @@
 	</joint>
 <!-- ======================================================== -->
-	<!-- Define joint between prop fl and frame -->
+<!-- Define joint between prop fl and frame -->
 	<joint name="joint_front_left_prop" type="continuous">
 		<parent link="base_link1" />
@@ -299,4 +413,36 @@
 	</joint>
 <!-- ======================================================== -->
+<!-- Define joint between prop fm and frame -->
+	<joint name="joint_front_middle_prop" type="continuous">
+		<parent link="base_link3" />
+		<child link="prop_front_middle" />
+		<origin xyz="0 ${prop_loc - 0.01} 0.021" rpy="0 0 ${pi_value/2}"/>
+		<axis xyz="0 0 1" />
+	</joint>
+<!-- ======================================================== -->
+<!-- Define joint between prop bm and frame -->
+	<joint name="joint_back_middle_prop" type="continuous">
+		<parent link="base_link3" />
+		<child link="prop_back_middle" />
+		<origin xyz="0 ${-prop_loc + 0.01} 0.021" rpy="0 0 ${-pi_value/2}" />
+		<axis xyz="0 0 1" />
+	</joint>
+<!-- ======================================================== -->
+<!-- Define joint between prop rm and frame -->
+	<joint name="joint_right_middle_prop" type="continuous">
+		<parent link="base_link4" />
+		<child link="prop_right_middle" />
+		<origin xyz="${prop_loc - 0.01} 0 0.021" rpy="0 0 0" />
+		<axis xyz="0 0 1" />
+	</joint>
+<!-- ======================================================== -->
+<!-- Define joint between prop lm and frame -->
+	<joint name="joint_left_middle_prop" type="continuous">
+		<parent link="base_link4" />
+		<child link="prop_left_middle" />
+		<origin xyz="${-prop_loc + 0.01} 0 0.021" rpy="0 0 0" />
+		<axis xyz="0 0 1" />
+	</joint>
+<!-- ======================================================== -->
 <!-- Define joint between plate1 and frame -->
 	<joint name="joint_plate1_frame" type="fixed">
@@ -404,3 +550,43 @@
 		</actuator>
 	</transmission>
+	<transmission name="front_middle_motor_joint" >
+		<type>transmission_interface/SimpleTransmission</type>
+		<joint name="joint_front_middle_prop">
+			<hardwareInterface>hardware_interface/VelocityJointInterface</hardwareInterface>
+		</joint>
+		<actuator name="BLDC_motor5">
+			<hardwareInterface>hardware_interface/VelocityJointInterface</hardwareInterface>
+			<mechanicalReduction>1</mechanicalReduction>
+		</actuator>
+	</transmission>
+	<transmission name="back_middle_motor_joint" >
+		<type>transmission_interface/SimpleTransmission</type>
+		<joint name="joint_back_middle_prop">
+			<hardwareInterface>hardware_interface/VelocityJointInterface</hardwareInterface>
+		</joint>
+		<actuator name="BLDC_motor6">
+			<hardwareInterface>hardware_interface/VelocityJointInterface</hardwareInterface>
+			<mechanicalReduction>1</mechanicalReduction>
+		</actuator>
+	</transmission>
+	<transmission name="right_middle_motor_joint" >
+		<type>transmission_interface/SimpleTransmission</type>
+		<joint name="joint_right_middle_prop">
+			<hardwareInterface>hardware_interface/VelocityJointInterface</hardwareInterface>
+		</joint>
+		<actuator name="BLDC_motor7">
+			<hardwareInterface>hardware_interface/VelocityJointInterface</hardwareInterface>
+			<mechanicalReduction>1</mechanicalReduction>
+		</actuator>
+	</transmission>
+	<transmission name="left_middle_motor_joint" >
+		<type>transmission_interface/SimpleTransmission</type>
+		<joint name="joint_left_middle_prop">
+			<hardwareInterface>hardware_interface/VelocityJointInterface</hardwareInterface>
+		</joint>
+		<actuator name="BLDC_motor8">
+			<hardwareInterface>hardware_interface/VelocityJointInterface</hardwareInterface>
+			<mechanicalReduction>1</mechanicalReduction>
+		</actuator>
+	</transmission>
 </robot>

Commit message: updated xacro file to rotate the propellers 90 degrees to match the design of last semesters robot

File: 2020_workspace/src/mate_simulation/urdf/Kwad.xacro (robot description, xacro)
@@ -385,5 +385,5 @@
 		<parent link="base_link2" />
 		<child link="prop_front_right" />
-		<origin xyz="${prop_loc - 0.01} ${prop_loc - 0.01} 0.021" rpy="${pi_value/2} 0 ${-pi_value/4}"/>
+		<origin xyz="${prop_loc - 0.01} ${prop_loc - 0.01} 0.021" rpy="${pi_value/2} 0 ${pi_value/4}"/>
 		<axis xyz="0 0 1" />
 	</joint>
@@ -393,5 +393,5 @@
 		<parent link="base_link1" />
 		<child link="prop_front_left" />
-		<origin xyz="${-prop_loc + 0.01} ${prop_loc - 0.01} 0.021" rpy="${pi_value/2} 0 ${pi_value/4}" />
+		<origin xyz="${-prop_loc + 0.01} ${prop_loc - 0.01} 0.021" rpy="${pi_value/2} 0 ${-pi_value/4}" />
 		<axis xyz="0 0 1" />
 	</joint>
@@ -401,13 +401,13 @@
 		<parent link="base_link1" />
 		<child link="prop_back_right" />
-		<origin xyz="${prop_loc - 0.01} ${-prop_loc + 0.01} 0.021" rpy="${pi_value/2} 0 ${pi_value/4}" />
-		<axis xyz="0 0 1" />
-	</joint>
-<!-- ======================================================== -->
-<!-- Define joint between prop br and frame -->
+		<origin xyz="${prop_loc - 0.01} ${-prop_loc + 0.01} 0.021" rpy="${pi_value/2} 0 ${-pi_value/4}" />
+		<axis xyz="0 0 1" />
+	</joint>
+<!-- ======================================================== -->
+<!-- Define joint between prop bl and frame -->
 	<joint name="joint_back_left_prop" type="continuous">
 		<parent link="base_link2" />
 		<child link="prop_back_left" />
-		<origin xyz="${-prop_loc + 0.01} ${-prop_loc + 0.01} 0.021" rpy="${-pi_value/2} 0 ${-pi_value/4}" />
+		<origin xyz="${-prop_loc + 0.01} ${-prop_loc + 0.01} 0.021" rpy="${-pi_value/2} 0 ${pi_value/4}" />
 		<axis xyz="0 0 1" />
 	</joint>

Commit message: reduced mass of drone to allow it to float instead of sink

File: 2020_workspace/src/mate_simulation/urdf/Kwad.xacro (robot description, xacro)
@@ -5,6 +5,8 @@
 	<xacro:property name="length" value="0.45" />
 	<xacro:property name="height" value="0.01" />
-	<xacro:property name="mass_fr" value="0.5" />
-	<xacro:property name="mass_pr" value="0.0055" />
+	<xacro:property name="mass_fr" value="0.005" />
+	<!-- <xacro:property name="mass_fr" value="0.5" />
+	<xacro:property name="mass_pr" value="0.0055" /> -->
+	<xacro:property name="mass_pr" value="0.00055" />
 	<xacro:property name="pi_value" value="3.14159263" />
 	<xacro:property name="radiusp" value="0.20" />

Commit message: very slighty neutrally bouyant drone.

File: 2020_workspace/src/mate_simulation/urdf/Kwad.xacro (robot description, xacro)
@@ -5,5 +5,5 @@
 	<xacro:property name="length" value="0.45" />
 	<xacro:property name="height" value="0.01" />
-	<xacro:property name="mass_fr" value="0.005" />
+	<xacro:property name="mass_fr" value="0.1755" />
 	<!-- <xacro:property name="mass_fr" value="0.5" />
 	<xacro:property name="mass_pr" value="0.0055" /> -->

Commit message: updated mass of drone to make it neutrally buoyant (almost). set color of front propeller to golden so it is different from other propellers. rotated 2 propellers so their joints are similar to the rest of the propellers.

File: 2020_workspace/src/mate_simulation/urdf/Kwad.xacro (robot description, xacro)
@@ -5,8 +5,7 @@
 	<xacro:property name="length" value="0.45" />
 	<xacro:property name="height" value="0.01" />
-	<xacro:property name="mass_fr" value="0.1755" />
-	<!-- <xacro:property name="mass_fr" value="0.5" />
-	<xacro:property name="mass_pr" value="0.0055" /> -->
-	<xacro:property name="mass_pr" value="0.00055" />
+	<xacro:property name="mass_fr" value="0.165" />
+	<xacro:property name="mass_pr" value="0.0055" />
+	<!-- <xacro:property name="mass_fr" value="0.5" /> -->
 	<xacro:property name="pi_value" value="3.14159263" />
 	<xacro:property name="radiusp" value="0.20" />
@@ -300,5 +299,5 @@
 				<box size="${0.03302/3} ${radiusp*0.8} ${0.001}" />
 			</geometry>
-			<material name="black" />
+			<material name="golden" />
 		</visual>
 		<collision>
@@ -395,5 +394,5 @@
 		<parent link="base_link1" />
 		<child link="prop_front_left" />
-		<origin xyz="${-prop_loc + 0.01} ${prop_loc - 0.01} 0.021" rpy="${pi_value/2} 0 ${-pi_value/4}" />
+		<origin xyz="${-prop_loc + 0.01} ${prop_loc - 0.01} 0.021" rpy="${pi_value/2} 0 ${3*pi_value/4}" />
 		<axis xyz="0 0 1" />
 	</joint>
@@ -443,5 +442,5 @@
 		<parent link="base_link4" />
 		<child link="prop_left_middle" />
-		<origin xyz="${-prop_loc + 0.01} 0 0.021" rpy="0 0 0" />
+		<origin xyz="${-prop_loc + 0.01} 0 0.021" rpy="0 0 ${pi_value}" />
 		<axis xyz="0 0 1" />
 	</joint>
