Commit message: Completed controllable ROV yaw,pitch,roll,forward/reverse,up/down, trucking left/right.

File: 2020_workspace/src/mate_simulation/urdf/rov.xacro (robot description, xacro)
@@ -1,4 +1,4 @@
 <?xml version="1.0"?>
-<robot xmlns:xacro="http://www.ros.org/wiki/xacro" name="Kwad">
+<robot xmlns:xacro="http://www.ros.org/wiki/xacro" name="rov">
 <!-- ======================================================== -->
 	<xacro:property name="width" value="0.0315" />
@@ -12,6 +12,6 @@
 	<xacro:property name="prop_loc" value="0.15909" />
 <!-- ======================================================== -->
-	<xacro:include filename="$(find fly_bot)/urdf/material.xacro" />
-	<xacro:include filename="$(find fly_bot)/urdf/Kwad.gazebo" />
+	<xacro:include filename="$(find mate_simulation)/urdf/material.xacro" />
+	<xacro:include filename="$(find mate_simulation)/urdf/rov.gazebo" />
 <!-- ======================================================== -->
 	<!-- Define inertial macro -->
@@ -199,5 +199,5 @@
 			<origin xyz="0 0 0" rpy="0 0 0" />
 			<geometry>
-				<mesh filename="package://fly_bot/meshes/22V10.dae" scale="0.005 0.005 0.005" />
+				<mesh filename="package://mate_simulation/meshes/22V10.dae" scale="0.005 0.005 0.005" />
 			</geometry>
 		</visual>
